Commit message: Added the gazebo plugins

File: src/buddy_description/urdf/gazebo_physics.xacro (robot description, xacro)
@@ -1,3 +1,112 @@
 <?xml version="1.0"?>
 <robot xmlns:xacro="http://www.ros.org/wiki/xacro" name="buddy">
+    <xacro:property name="standard_friction" value="1.0" />
+    <xacro:property name="caster_friction" value="0.01" />
+    <xacro:property name="wheels_friction" value="1000.0" />
+    <gazebo reference="base_link">
+    <mu1>${standard_friction}</mu1>
+    <mu2>${standard_friction}</mu2>
+    <selfCollide>true</selfCollide>
+    <gravity>true</gravity>
+    </gazebo>
+    <gazebo reference="right_wheel">
+    <mu1>${standard_friction}</mu1>
+    <mu2>${standard_friction}</mu2>
+    <selfCollide>true</selfCollide>
+    </gazebo>
+    <gazebo reference="left_wheel">
+    <mu1>${standard_friction}</mu1>
+    <mu2>${standard_friction}</mu2>
+    <selfCollide>true</selfCollide>
+    </gazebo>
+    <gazebo reference="right_tyre">
+    <mu1>${wheels_friction}</mu1>
+    <mu2>${wheels_friction}</mu2>
+    <selfCollide>true</selfCollide>
+    </gazebo>
+    <gazebo reference="left_tyre">
+    <mu1>${wheels_friction}</mu1>
+    <mu2>${wheels_friction}</mu2>
+    <selfCollide>true</selfCollide>
+    </gazebo>
+    <gazebo reference="front_caster">
+    <mu1>${caster_friction}</mu1>
+    <mu2>${caster_friction}</mu2>
+    <selfCollide>true</selfCollide>
+    </gazebo>
+    <gazebo reference="back_caster">
+    <mu1>${caster_friction}</mu1>
+    <mu2>${caster_friction}</mu2>
+    <selfCollide>true</selfCollide>
+    </gazebo>
+    <gazebo reference="lid">
+    <mu1>${standard_friction}</mu1>
+    <mu2>${standard_friction}</mu2>
+    <selfCollide>true</selfCollide>
+    </gazebo>
+    <gazebo reference="lidar">
+    <mu1>${standard_friction}</mu1>
+    <mu2>${standard_friction}</mu2>
+    <selfCollide>true</selfCollide>
+    </gazebo>
+    <gazebo reference="electronics_lid">
+    <mu1>${standard_friction}</mu1>
+    <mu2>${standard_friction}</mu2>
+    <selfCollide>true</selfCollide>
+    </gazebo>
+    <gazebo reference="long_bar">
+    <mu1>${standard_friction}</mu1>
+    <mu2>${standard_friction}</mu2>
+    <selfCollide>true</selfCollide>
+    </gazebo>
+    <gazebo reference="head">
+    <mu1>${standard_friction}</mu1>
+    <mu2>${standard_friction}</mu2>
+    <selfCollide>true</selfCollide>
+    </gazebo>
+    <gazebo reference="visor">
+    <mu1>${standard_friction}</mu1>
+    <mu2>${standard_friction}</mu2>
+    <selfCollide>true</selfCollide>
+    </gazebo>
+    <gazebo reference="monitor_cover">
+    <mu1>${standard_friction}</mu1>
+    <mu2>${standard_friction}</mu2>
+    <selfCollide>true</selfCollide>
+    </gazebo>
+    <gazebo reference="right_ear">
+    <mu1>${standard_friction}</mu1>
+    <mu2>${standard_friction}</mu2>
+    <selfCollide>true</selfCollide>
+    </gazebo>
+    <gazebo reference="left_ear">
+    <mu1>${standard_friction}</mu1>
+    <mu2>${standard_friction}</mu2>
+    <selfCollide>true</selfCollide>
+    </gazebo>
+    <gazebo reference="monitor">
+    <mu1>${standard_friction}</mu1>
+    <mu2>${standard_friction}</mu2>
+    <selfCollide>true</selfCollide>
+    </gazebo>
+    <gazebo reference="left_antenna">
+    <mu1>${standard_friction}</mu1>
+    <mu2>${standard_friction}</mu2>
+    <selfCollide>true</selfCollide>
+    </gazebo>
+    <gazebo reference="right_antenna">
+    <mu1>${standard_friction}</mu1>
+    <mu2>${standard_friction}</mu2>
+    <selfCollide>true</selfCollide>
+    </gazebo>
+    <gazebo reference="camera_link">
+    <mu1>${standard_friction}</mu1>
+    <mu2>${standard_friction}</mu2>
+    <selfCollide>true</selfCollide>
+    </gazebo>
+    <gazebo reference="realsense">
+    <mu1>${standard_friction}</mu1>
+    <mu2>${standard_friction}</mu2>
+    <selfCollide>true</selfCollide>
+    </gazebo>
 </robot>

File: src/buddy_description/urdf/gazebo_plugins.xacro (robot description, xacro)
@@ -1,3 +1,64 @@
 <?xml version="1.0"?>
 <robot xmlns:xacro="http://www.ros.org/wiki/xacro" name="buddy">
+    <!-- ############# ROS CONTROL ############# -->
+    <gazebo>
+    <plugin filename="libgazebo_ros_control.so" name="control"/>
+    </gazebo>
+    <!-- ############# DIFFERENTIAL DRIVE ############# -->
+    <gazebo>
+    <plugin name="differential_drive_controller" filename="libgazebo_ros_diff_drive.so">
+        <updateRate>20</updateRate>
+        <leftJoint>motor_left</leftJoint>
+        <rightJoint>motor_right</rightJoint>
+        <wheelSeparation>0.36</wheelSeparation>
+        <wheelDiameter>0.20</wheelDiameter>
+        <wheelAcceleration>1.0</wheelAcceleration>
+        <wheelTorque>20</wheelTorque>
+        <commandTopic>cmd_vel</commandTopic>
+        <odometryTopic>odom</odometryTopic>
+        <odometryFrame>odom</odometryFrame>
+        <robotBaseFrame>base_link</robotBaseFrame>
+        <odometrySource>1</odometrySource>
+        <publishWheelTF>true</publishWheelTF>
+        <publishOdom>true</publishOdom>
+        <publishWheelJointState>true</publishWheelJointState>
+        <legacyMode>false</legacyMode>
+    </plugin>
+    </gazebo>
+    <!-- ############# LIDAR PLUGIN ############# -->
+    <gazebo reference="lidar">
+        <sensor type="ray" name="rplidar_a1">
+        <pose>0 0 0 0 0 0</pose>
+        <visualize>false</visualize>
+        <update_rate>10</update_rate>
+        <ray>
+            <scan>
+            <horizontal>
+                <samples>720</samples>
+                <resolution>1</resolution>
+                <min_angle>-2.87979</min_angle>
+                <max_angle>2.87979</max_angle>
+            </horizontal>
+            </scan>
+            <range>
+            <min>0.10</min>
+            <max>20.0</max>
+            <resolution>0.01</resolution>
+            </range>
+            <noise>
+            <type>gaussian</type>
+            <!-- Noise parameters based on published spec for Hokuyo laser
+                achieving "+-30mm" accuracy at range < 10m.  A mean of 0.0m and
+                stddev of 0.01m will put 99.7% of samples within 0.03m of the true
+                reading. -->
+            <mean>0.0</mean>
+            <stddev>0.01</stddev>
+            </noise>
+        </ray>
+        <plugin name="gazebo_ros_head_hokuyo_controller" filename="libgazebo_ros_laser.so">
+            <topicName>/scan</topicName>
+            <frameName>lidar</frameName>
+        </plugin>
+        </sensor>
+    </gazebo>
 </robot>
